File: Harwdare/Pet-Feeder/Pet-Feeder.kicad_sch (KiCad schematic)
At the start: 19 parts

Commit message: Comecei a separar como eu quero que o codigo esteja
Connections:
- net CONTROL: now also U?.30 (IO18); no longer U?.16 (IO13)
Changed lines of the file:
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@@
     )
   )
-  (global_label "CONTROL" (shape output) (at 215.9 69.088 0) (fields_autoplaced)
+  (global_label "CONTROL" (shape output) (at 215.9 81.788 0) (fields_autoplaced)
     (effects (font (size 1.27 1.27)) (justify left))
-    (property "Intersheet References" "${INTERSHEET_REFS}" (id 0) (at 226.8402 69.0086 0)
+    (property "Intersheet References" "${INTERSHEET_REFS}" (id 0) (at 226.8402 81.7086 0)
       (effects (font (size 1.27 1.27)) (justify left) hide)
     )
